Commit message: imu and robot_localization

File: tortoisebot_description/models/urdf/tortoisebot_simple.xacro (robot description, xacro)
@@ -138,4 +138,23 @@
 </link>
 <link name="imu_link"/>
+<!-- <link name="imu"> -->
+  <inertial>
+    <origin xyz="0.0 0.0 0.0" rpy="0 0 0"/>
+    <mass value="0.001"/>
+    <inertia ixx="1e-06" iyy="1e-06" izz="1e-06" ixy="0.0" iyz="0.0" ixz="0.0"/>
+  </inertial>
+  <visual>
+      <geometry>
+          <box size="0.1 0.1 0.1" />
+      </geometry>
+      <material name="Cyan">
+          <color rgba="0 1.0 1.0 1.0" />
+      </material>
+  </visual>
+  <collision>
+      <geometry>
+          <box size="0.1 0.1 0.1" />
+      </geometry>
+  </collision>
 <joint name="wheel_left_joint" type="continuous">
   <origin xyz="-0.000197 0.0778 0.032453" rpy="0 0 0"/>
